File: hardware/ttl_io/ttl_io.kicad_pcb (KiCad board)
At the start: 4 copper layers, 120 x 75 mm, 198 parts, among them J1 Conn_01x03_Male, J10 Conn_Coaxial, J11 Conn_Coaxial, J12 Conn_Coaxial, J13 Conn_02x08_Counter_Clockwise, J14 Conn_02x08_Counter_Clockwise, J2 AudioJack3, J3 USB_C_Receptacle_USB2.0, J4 Barrel_Jack_Switch, J5 Conn_Coaxial, J6 Conn_Coaxial, J7 Conn_Coaxial, J8 Conn_Coaxial, J9 Conn_Coaxial, SW1 SW_Push, SW2 SW_SPDT, SW3 SW_SPDT, U1 TPD2EUSB30, U10 74LVCH2T45DC, U11 74LVCH2T45DC, U12 74LVCH2T45DC, U13 74LVCH2T45DC, U14 74CBTLV3245, U15 SN74LVC1G14DRL, U16 74CBTLV3245, U17 74CBTLV3245, U18 SN74LVC1G14DRL, U19 TXB0108, U2 ADUM4160, U3 RP2040, U4 W25Q16JVUXIQ, U5 74LVCH2T45DC, U6 74LVCH2T45DC, U7 74LVCH2T45DC, U8 LT3506, U9 74LVCH2T45DC, X1 ECS-TXO-2016

Commit message: draft pcb v0.1.0
Parts:
- removed the C7 at (171.9, 78.2)
- removed the C9 at (170.8, 83.2)
- added G***: LOGO, LOGO, B.Cu at (186.9, 80.5)
- J10, J11, J12, J5, J6, J7, J8, J9: moved to F.Cu
- J4: footprint Connector_BarrelJack:BarrelJack_CUI_PJ-036AH-SMT_Horizontal -> Connector_BarrelJack:BarrelJack_CUI_PJ-102AH_Horizontal
- SW1: value SW_Push -> ~; footprint Button_Switch_SMD:SW_SPST_B3U-1000P -> kicad_component_library:SW_Push_1P1T-SH_NO_Vertical_Wuerth_WS-TASV
- moved C81 22.5 mm to (195.1, 63.0), turned to -90 degrees
- moved R44 21.5 mm to (197.1, 63.0), turned to 90 degrees
- moved C79 20.5 mm to (196.1, 63.0), turned to 90 degrees
- moved R48 18.7 mm to (198.1, 63.0), turned to -90 degrees
- moved U18 18.4 mm to (196.3, 60.7), turned to 180 degrees
- moved C77 16.2 mm to (199.1, 63.0), turned to 90 degrees
- moved U15 16.0 mm to (199.3, 60.7), turned to 180 degrees
- moved C78 15.9 mm to (201.0, 60.7)
- moved C80 15.9 mm to (202.0, 60.7)
- moved R43 15.9 mm to (203.0, 60.7)
- moved C62 15.9 mm to (133.7, 71.8), turned to 0 degrees
- moved C63 14.3 mm to (133.7, 72.8)
- moved C76 13.7 mm to (178.6, 62.3)
- moved D11 13.7 mm to (177.1, 60.8)
- moved R47 13.7 mm to (178.6, 60.3)
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Connections:
- SW1 pad 1: GND -> unconnected-(SW1-Pad1)
Routing:
- net /TTL_DIR0: track 0.00 -> 94.6 mm, vias 0 -> 2
- net /TTL7: track 6.36 -> 85.8 mm, vias 0 -> 2
- net /TTL_DIR3: track 7.92 -> 76.9 mm, vias 0 -> 2
- net /TTL0: track 10.7 -> 75.6 mm, vias 0 -> 2
- net /TTL_DIR1: track 6.84 -> 69.7 mm, vias 0 -> 2
- net /TTL_DIR7: track 10.1 -> 72.9 mm, vias 0 -> 2
- net /TTL6: track 6.90 -> 67.1 mm, vias 0 -> 2
- net /TTL_DIR2: track 7.38 -> 65.7 mm, vias 0 -> 2
- net /TTL5: track 7.43 -> 64.5 mm, vias 0 -> 2
- net /TTL4: track 7.97 -> 64.7 mm, vias 0 -> 2
- net /TTL_DIR6: track 9.55 -> 50.6 mm, vias 0 -> 2
- net GND: track 64.4 -> 104.1 mm, vias 57 -> 79
- net /TTL1: track 11.2 -> 45.3 mm, vias 1 -> 2
- net +5V: track 29.4 -> 63.5 mm, vias 4 -> 14
- net /TTL2: track 9.59 -> 42.4 mm, vias 0 -> 2
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Other:
- board text added: "0"
- board text added: "1"
- board text added: "2"
- board text added: "3"
- board text added: "4"
- board text added: "5"
- board text added: "6"
- board text added: "7"
- board text added: "Ext I/O mode: TTL inputs/outputs controlled by pins on the board edge. (Orange LED On.) USB I/O mode: TTL inputs/outputs controlled by software over USB interface. (Orange LED Off.)"
- board text added: "External Input Logic Level Selection"
- board text added: "_____DIR (Top Row)_____ | |"
- board text added: "______IO (Top Row)_____ | |"
- board text added: "v0.1.0, Jan 4, 2024"
- board text added: "|___GND (Bottom Row)____|"
- board text added: "▪"
- board text removed: "CuTTLfish can be used in two ways: 1.) as a programmable square wave generator with 8 TTL outputs. 2.) as a TTl buffer for 3.3V logic (input and output)"
- board text removed: "Ext I/O mode: TTL input/output controlled by pins on the board edge. (Orange LED On.) USB I/O mode: TTL input/output controlled by software over USB interface. (Orange LED Off.)"
- board text removed: "External Input Logic Level Selection Switch"
- board text removed: "TODO: Connector heights. * Put everything on top except the BNC connectors?"
- board text removed: "TODO: Switch BOOTSEL switch for washable variant."
- board text removed: "v0.1.0, Jan 3, 2024"

Commit message: update pcb and bom
Parts:
- G3: moved to F.Cu
- J10, J11, J12, J5, J6, J7, J8, J9: footprint kicad_component_library:BNC_TEConnectivity_CONBNC001_Vertical -> kicad_component_library:BNC_AmphenolRF_031-5329-52RFX_Vertical
- J4: moved to B.Cu
- moved G3 5.00 mm to (222.4, 96.0), turned to -90 degrees
- turned J4 to -90 degrees
Routing:
- net Net-(D9-A): track 28.0 -> 26.0 mm, vias 0 -> 2
- net GND2: track 17.8 -> 16.4 mm
- net ~{HARP_CTRL}: track 54.4 -> 55.0 mm
Other:
- board text added: "v0.1.0, Jan 11, 2024"
- board text removed: "Hammond: 1455J1202BK"
- board text removed: "v0.1.0, Jan 4, 2024"

Commit message: draft scheduler
Connections:
- J13 pad 10: /EXT_DIR6 -> /EXT_DIR1
- J13 pad 11: /EXT_DIR5 -> /EXT_DIR2
- J13 pad 12: /EXT_DIR4 -> /EXT_DIR3
- J13 pad 13: /EXT_DIR3 -> /EXT_DIR4
- J13 pad 14: /EXT_DIR2 -> /EXT_DIR5
- J13 pad 15: /EXT_DIR1 -> /EXT_DIR6
- J13 pad 16: /EXT_DIR0 -> /EXT_DIR7
- J13 pad 9: /EXT_DIR7 -> /EXT_DIR0
- J14 pad 10: /EXT_IN6 -> /EXT_IN1
- J14 pad 11: /EXT_IN5 -> /EXT_IN2
- J14 pad 12: /EXT_IN4 -> /EXT_IN3
- J14 pad 13: /EXT_IN3 -> /EXT_IN4
- J14 pad 14: /EXT_IN2 -> /EXT_IN5
- J14 pad 15: /EXT_IN1 -> /EXT_IN6
- J14 pad 16: /EXT_IN0 -> /EXT_IN7
- J14 pad 9: /EXT_IN7 -> /EXT_IN0
Other:
- board text added: "v0.1.1, Jan 16, 2024"
- board text removed: "v0.1.0, Jan 11, 2024"
