File: hardware/ttl_io/power_supplies.kicad_sch (KiCad schematic)
At the start: 22 parts, among them J5 Barrel_Jack_Switch, U8 LT3506

Commit message: draft mcu bypass with bus switches
Parts:
- removed R23: 15K, symbol Device:R
- added D8: D_Schottky, Diode_SMD:D_SOD-123, symbol Device:D_Schottky
- added R8: 10K, Resistor_SMD:R_0402_1005Metric, symbol Device:R
- C33: footprint (none) -> Resistor_SMD:R_0402_1005Metric; Link (none) -> https://www.digikey.com/en/products/detail/yageo/CC0402KRX7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; Manufacturer (none) -> Yageo; Manufacturer Number (none) -> CC0402KRX7R9BB152; Temperature Coefficient (none) -> X7R; Tolerance (none) -> 10%; Voltage Rating (none) -> 50V
- C34: footprint (none) -> Resistor_SMD:R_0402_1005Metric; Link (none) -> https://www.digikey.com/en/products/detail/murata-electroni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; Manufacturer (none) -> Murata Electronics; Manufacturer Number (none) -> GCM155R71H472KA37J; Temperature Coefficient (none) -> X7R; Tolerance (none) -> 10%; Voltage Rating (none) -> 50V
- C35: footprint (none) -> Resistor_SMD:R_0402_1005Metric; Link (none) -> https://www.digikey.com/en/products/detail/yageo/CC0402KRX7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; Manufacturer (none) -> Yageo; Manufacturer Number (none) -> CC0402KRX7R9BB152; Temperature Coefficient (none) -> X7R; Tolerance (none) -> 10%
- D5: Link (none) -> https://www.digikey.com/en/products/detail/diodes-incorpora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; Manufacturer (none) -> Diodes Incorporated; Manufacturer Number (none) -> BAT54AW-7-F
- D6, D7: footprint (none) -> Diode_SMD:D_SMA; Link (none) -> https://www.digikey.com/en/products/detail/smc-diode-soluti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; Manufacturer (none) -> SMC Diode Solutions; Manufacturer Number (none) -> SL13
- L2, L3: value 2.2uH -> 10uH; footprint (none) -> Inductor_SMD:L_Vishay_IHLP-2525; Link https://www.digikey.com/en/products/detail/coilcraft/LPS401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 -> https://www.digikey.com/en/products/detail/vishay-dale/IHLP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
- R24: footprint (none) -> Resistor_SMD:R_0402_1005Metric; Link (none) -> https://www.digikey.com/en/products/detail/koa-speer-electr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; Manufacturer (none) -> KOA Speer Electronics, Inc.; Manufacturer Number (none) -> RN73H1ETTP3122F25; Tolerance (none) -> 1%
- R26: value 52K5 -> 52K3; footprint (none) -> Resistor_SMD:R_0402_1005Metric; Link (none) -> https://www.digikey.com/en/products/detail/yageo/RT0402FRE0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; Manufacturer (none) -> Yageo; Manufacturer Number (none) -> RT0402FRE0752K3L; Tolerance (none) -> 1%
Connections:
- net +12V: now also D8.2 (A); no longer L1.2
- net GND: now also R8.1
- net at C35.2: now also R8.2
- new net: D8.1 (K), L1.2
Other:
- note added: "LT3506 Datasheet: feedback resistors in parallel (i.e: R21||R24 and R25||R26) should be less than 10K."
- note added: "Reverse Polarity Protection"
- note added: "Warning: The above configuration is not interchangeable with the LT3506A."
- note removed: "FIXME: Inductors might need to be closer to 10uH"
- note removed: "LT3506 Datasheet: feedback resistors in parallel (R21||R24 and R25||R26) should be less than 10K."
- note removed: "Warning: Not interchangeable with the LT3506A."
- moved on the sheet: C37, J5, L1

Commit message: update passthrough level translator
Parts:
- D6, D7: footprint Diode_SMD:D_SMA -> Diode_SMD:D_SOD-123; Link https://www.digikey.com/en/products/detail/smc-diode-solutions/SL13/5993518 -> https://www.digikey.com/en/products/detail/smc-diode-solutions/MBR260HW/5993805; Manufacturer SMC Diode Solutions -> (none); Manufacturer Number SL13 -> MBR260HW
- J4: renamed from J5; footprint Connector_BarrelJack:BarrelJack_CUI_PJ-102AH_Horizontal -> Connector_BarrelJack:BarrelJack_CUI_PJ-036AH-SMT_Horizontal; Link https://www.digikey.com/en/products/detail/cui-devices/PJ-1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 -> https://www.digikey.com/en/products/detail/cui-devices/PJ-0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; Manufacturer Number PJ-102AH -> PJ-036AH-SMT-TR; PCBWay Link https://www.pcbway.com/components/detail/PJ102AH/484087/ -> https://www.pcbway.com/components/detail/PJ036AHSMTTR/39245/
- U8: Manufacturer (none) -> Analog Devices Inc.; Manufacturer Number (none) -> LT3506EDHD#PBF
Changed lines of the file:
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@@
-    )
-  )
-  (symbol (lib_id "Device:D_Schottky") (at 119.38 100.965 90) (mirror x) (unit 1)
-    (in_bom yes) (on_board yes) (dnp no)
-    (property "Reference" "D7" (at 118.745 97.79 90)
-      (effects (font (size 1.27 1.27)) (justify left))
-    )
-    (property "Value" "D_Schottky" (at 116.205 101.9175 90)
-      (effects (font (size 1.27 1.27)) (justify left) hide)
-    )
-    (property "Footprint" "Diode_SMD:D_SMA" (at 119.38 100.965 0)
-      (effects (font (size 1.27 1.27)) hide)
-    )
-    (property "Datasheet" "~" (at 119.38 100.965 0)
-      (effects (font (size 1.27 1.27)) hide)
-    )
-    (property "Link" "https://www.digikey.com/en/products/detail/smc-diode-solutions/SL13/5993518" (at 119.38 100.965 90)
-      (effects (font (size 1.27 1.27)) hide)
-    )
-    (property "Manufacturer" "SMC Diode Solutions" (at 119.38 100.965 90)
-      (effects (font (size 1.27 1.27)) hide)
-    )
-    (property "Manufacturer Number" "SL13" (at 119.38 100.965 90)
-      (effects (font (size 1.27 1.27)) hide)
-    )
-    (pin "1")
-    (pin "2")
-    (instances
-      (project "ttl_io"
-        (path "/de782c9d-fd54-45ed-aa91-6297331e40f6/76bb2607-2d2e-4d2c-9a45-1b3b3938988a"
-          (reference "D7") (unit 1)
-        )
-      )
     )
   )
@@
   (symbol (lib_id "Connector:Barrel_Jack_Switch") (at 29.845 69.85 0) (unit 1)
     (in_bom yes) (on_board yes) (dnp no)
-    (property "Reference" "J5" (at 26.035 64.77 0)
+    (property "Reference" "J4" (at 26.035 64.77 0)
       (effects (font (size 1.27 1.27)))
     )
@@
       (effects (font (size 1.27 1.27)) hide)
     )
-    (property "Footprint" "Connector_BarrelJack:BarrelJack_CUI_PJ-102AH_Horizontal" (at 31.115 70.866 0)
-      (effects (font (size 1.27 1.27)) hide)
-    )
-    (property "Datasheet" "https://www.cuidevices.com/product/resource/pj-102ah.pdf" (at 31.115 70.866 0)
-      (effects (font (size 1.27 1.27)) hide)
-    )
-    (property "Link" "https://www.digikey.com/en/products/detail/cui-devices/PJ-102AH/408448" (at 29.845 69.85 0)
-      (effects (font (size 1.27 1.27)) hide)
-    )
-    (property "Manufacturer Number" "PJ-102AH" (at 29.845 69.85 0)
-      (effects (font (size 1.27 1.27)) hide)
-    )
-    (property "PCBWay Link" "https://www.pcbway.com/components/detail/PJ102AH/484087/" (at 29.845 69.85 0)
+    (property "Footprint" "Connector_BarrelJack:BarrelJack_CUI_PJ-036AH-SMT_Horizontal" (at 31.115 70.866 0)
+      (effects (font (size 1.27 1.27)) hide)
+    )
+    (property "Datasheet" "https://www.cuidevices.com/product/resource/pj-036ah-smt-tr.pdf" (at 31.115 70.866 0)
+      (effects (font (size 1.27 1.27)) hide)
+    )
+    (property "Link" "https://www.digikey.com/en/products/detail/cui-devices/PJ-036AH-SMT-TR/1530994?" (at 29.845 69.85 0)
+      (effects (font (size 1.27 1.27)) hide)
+    )
+    (property "Manufacturer Number" "PJ-036AH-SMT-TR" (at 29.845 69.85 0)
+      (effects (font (size 1.27 1.27)) hide)
+    )
+    (property "PCBWay Link" "https://www.pcbway.com/components/detail/PJ036AHSMTTR/39245/" (at 29.845 69.85 0)
       (effects (font (size 1.27 1.27)) hide)
     )
@@
       (project "ttl_io"
         (path "/de782c9d-fd54-45ed-aa91-6297331e40f6/76bb2607-2d2e-4d2c-9a45-1b3b3938988a"
-          (reference "J5") (unit 1)
+          (reference "J4") (unit 1)
         )
       )
@@
     )
   )
+  (symbol (lib_id "Device:D_Schottky") (at 178.435 100.965 270) (unit 1)
+    (in_bom yes) (on_board yes) (dnp no)
+    (property "Reference" "D6" (at 179.705 97.79 90)
+      (effects (font (size 1.27 1.27)))
+    )
+    (property "Value" "D_Schottky" (at 174.625 100.6475 0)
+      (effects (font (size 1.27 1.27)) hide)
+    )
+    (property "Footprint" "Diode_SMD:D_SOD-123" (at 178.435 100.965 0)
+      (effects (font (size 1.27 1.27)) hide)
+    )
+    (property "Datasheet" "~" (at 178.435 100.965 0)
+      (effects (font (size 1.27 1.27)) hide)
+    )
+    (property "Link" "https://www.digikey.com/en/products/detail/smc-diode-solutions/MBR260HW/5993805" (at 178.435 100.965 0)
+      (effects (font (size 1.27 1.27)) hide)
+    )
+    (property "Manufacturer Number" "MBR260HW" (at 178.435 100.965 0)
+      (effects (font (size 1.27 1.27)) hide)
+    )
+    (pin "1")
+    (pin "2")
+    (instances
+      (project "ttl_io"
+        (path "/de782c9d-fd54-45ed-aa91-6297331e40f6/76bb2607-2d2e-4d2c-9a45-1b3b3938988a"
+          (reference "D6") (unit 1)
+        )
+      )
+    )
+  )
+  (symbol (lib_id "Device:D_Schottky") (at 119.38 100.965 270) (unit 1)
+    (in_bom yes) (on_board yes) (dnp no)
+    (property "Reference" "D7" (at 117.475 97.79 90)
+      (effects (font (size 1.27 1.27)))
+    )
+    (property "Value" "D_Schottky" (at 115.57 100.6475 0)
+      (effects (font (size 1.27 1.27)) hide)
+    )
+    (property "Footprint" "Diode_SMD:D_SOD-123" (at 119.38 100.965 0)
+      (effects (font (size 1.27 1.27)) hide)
+    )
+    (property "Datasheet" "~" (at 119.38 100.965 0)
+      (effects (font (size 1.27 1.27)) hide)
+    )
+    (property "Link" "https://www.digikey.com/en/products/detail/smc-diode-solutions/MBR260HW/5993805" (at 119.38 100.965 0)
+      (effects (font (size 1.27 1.27)) hide)
+    )
+    (property "Manufacturer Number" "MBR260HW" (at 119.38 100.965 0)
+      (effects (font (size 1.27 1.27)) hide)
+    )
+    (pin "1")
+    (pin "2")
+    (instances
+      (project "ttl_io"
+        (path "/de782c9d-fd54-45ed-aa91-6297331e40f6/76bb2607-2d2e-4d2c-9a45-1b3b3938988a"
+          (reference "D7") (unit 1)
+        )
+      )
+    )
+  )
   (symbol (lib_id "power:+5V") (at 194.945 89.535 0) (unit 1)
     (in_bom yes) (on_board yes) (dnp no)
@@
     )
     (property "Link" "https://www.digikey.com/en/products/detail/analog-devices-inc/LT3506EDHD-PBF/1620038" (at 148.59 93.98 0)
+      (effects (font (size 1.27 1.27)) hide)
+    )
+    (property "Manufacturer" "Analog Devices Inc." (at 148.59 93.98 0)
+      (effects (font (size 1.27 1.27)) hide)
+    )
+    (property "Manufacturer Number" "LT3506EDHD#PBF" (at 148.59 93.98 0)
       (effects (font (size 1.27 1.27)) hide)
     )
@@
         )
       )
-    )
-  )
-  (symbol (lib_id "Device:D_Schottky") (at 178.435 100.965 90) (mirror x) (unit 1)
-    (in_bom yes) (on_board yes) (dnp no)
-    (property "Reference" "D6" (at 181.61 97.79 90)
-      (effects (font (size 1.27 1.27)) (justify left))
-    )
-    (property "Value" "D_Schottky" (at 175.26 101.9175 90)
-      (effects (font (size 1.27 1.27)) (justify left) hide)
-    )
-    (property "Footprint" "Diode_SMD:D_SMA" (at 178.435 100.965 0)
-      (effects (font (size 1.27 1.27)) hide)
-    )
-    (property "Datasheet" "~" (at 178.435 100.965 0)
-      (effects (font (size 1.27 1.27)) hide)
-    )
-    (property "Link" "https://www.digikey.com/en/products/detail/smc-diode-solutions/SL13/5993518" (at 178.435 100.965 90)
-      (effects (font (size 1.27 1.27)) hide)
-    )
-    (property "Manufacturer" "SMC Diode Solutions" (at 178.435 100.965 90)
-      (effects (font (size 1.27 1.27)) hide)
-    )
-    (property "Manufacturer Number" "SL13" (at 178.435 100.965 90)
-      (effects (font (size 1.27 1.27)) hide)
-    )
-    (pin "1")
-    (pin "2")
-    (instances
-      (project "ttl_io"
-        (path "/de782c9d-fd54-45ed-aa91-6297331e40f6/76bb2607-2d2e-4d2c-9a45-1b3b3938988a"
-          (reference "D6") (unit 1)
-        )
-      )

Commit message: update power supply schematic/board
Connections:
- net +3V3: now also R24.2; no longer R8.2
- net +5V: now also R26.2; no longer R8.1
- net GND: now also R8.1, R8.2; no longer R24.2, R26.1
- net at C35.1, U8.10 (VC2): now also U8.14 (PG1)
- net at R8.2, U8.9 (FB2): now also R26.1; no longer R26.2
- no-connect marks 3 -> 2
Other:
- note added: "LT3506 Feedback: R_{upper} = R_{lower}(V_{out}/0.8 - 1)"
- moved on the sheet: R24, R26, R8
Changed lines of the file:
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@@
   (junction (at 114.3 95.885) (diameter 0) (color 0 0 0 0)
   )
+  (junction (at 161.925 95.885) (diameter 0) (color 0 0 0 0)
+  )
   (junction (at 182.88 106.045) (diameter 0) (color 0 0 0 0)
   )
@@
   (no_connect (at 37.465 69.85))
   (no_connect (at 137.16 111.125))
-  (no_connect (at 160.02 111.125))
   (wire (pts (xy 135.255 106.045) (xy 137.16 106.045))
     (stroke (width 0) (type default))
@@
     (stroke (width 0) (type default))
   )
+  (wire (pts (xy 160.02 111.125) (xy 161.925 111.125))
+    (stroke (width 0) (type default))
+  )
   (wire (pts (xy 124.46 106.045) (xy 124.46 104.775))
     (stroke (width 0) (type default))
@@
     (stroke (width 0) (type default))
   )
+  (wire (pts (xy 161.925 95.885) (xy 163.83 95.885))
+    (stroke (width 0) (type default))
+  )
   (wire (pts (xy 114.3 104.775) (xy 114.3 106.045))
     (stroke (width 0) (type default))
@@
     (stroke (width 0) (type default))
   )
+  (wire (pts (xy 161.925 111.125) (xy 161.925 95.885))
+    (stroke (width 0) (type default))
+  )
   (wire (pts (xy 124.46 95.885) (xy 124.46 97.155))
     (stroke (width 0) (type default))
@@
     (stroke (width 0) (type default))
   )
-  (wire (pts (xy 160.02 95.885) (xy 163.83 95.885))
+  (wire (pts (xy 160.02 95.885) (xy 161.925 95.885))
     (stroke (width 0) (type default))
   )
@@
     (effects (font (size 1.27 1.27)) (justify left bottom))
   )
+  (text "LT3506 Feedback:\nR_{upper} = R_{lower}(V_{out}/0.8 - 1)"
+    (at 185.42 56.515 0)
+    (effects (font (size 1.27 1.27)) (justify left bottom))
+  )
   (text "Warning: The above configuration is not interchangeable with the LT3506A."
     (at 125.095 128.905 0)
@@
     )
   )
-  (symbol (lib_id "Device:R") (at 187.96 95.885 270) (unit 1)
+  (symbol (lib_id "Device:R") (at 182.88 100.965 180) (unit 1)
     (in_bom yes) (on_board yes) (dnp no)
-    (property "Reference" "R8" (at 186.055 93.345 90)
+    (property "Reference" "R8" (at 185.42 99.06 90)
       (effects (font (size 1.27 1.27)) (justify left))
     )
-    (property "Value" "10K" (at 186.055 95.885 90)
+    (property "Value" "10K" (at 182.88 99.06 90)
       (effects (font (size 1.27 1.27)) (justify left))
     )
-    (property "Footprint" "Resistor_SMD:R_0402_1005Metric" (at 187.96 94.107 90)
+    (property "Footprint" "Resistor_SMD:R_0402_1005Metric" (at 184.658 100.965 90)
       (effects (font (size 1.27 1.27)) hide)
     )
-    (property "Datasheet" "https://www.koaspeer.com/pdfs/SG73P.pdf" (at 187.96 95.885 0)
+    (property "Datasheet" "https://www.koaspeer.com/pdfs/SG73P.pdf" (at 182.88 100.965 0)
       (effects (font (size 1.27 1.27)) hide)
     )
-    (property "Link" "https://www.digikey.com/en/products/detail/koa-speer-electronics-inc/SG73P1EWTTP1002F/14316756" (at 187.96 95.885 90)
+    (property "Link" "https://www.digikey.com/en/products/detail/koa-speer-electronics-inc/SG73P1EWTTP1002F/14316756" (at 182.88 100.965 90)
       (effects (font (size 1.27 1.27)) hide)
     )
-    (property "Manufacturer" "KOA Speer Electronics, Inc." (at 187.96 95.885 0)
+    (property "Manufacturer" "KOA Speer Electronics, Inc." (at 182.88 100.965 0)
       (effects (font (size 1.27 1.27)) hide)
     )
-    (property "Manufacturer Number" "SG73P1EWTTP1002F" (at 187.96 95.885 0)
+    (property "Manufacturer Number" "SG73P1EWTTP1002F" (at 182.88 100.965 0)
       (effects (font (size 1.27 1.27)) hide)
     )
-    (property "Notes" "DNP" (at 187.96 95.885 0)
+    (property "Notes" "DNP" (at 182.88 100.965 0)
       (effects (font (size 1.27 1.27)) hide)
     )
@@
     )
   )
-  (symbol (lib_id "Device:R") (at 114.3 100.965 0) (unit 1)
+  (symbol (lib_id "Device:R") (at 109.22 95.885 270) (unit 1)
     (in_bom yes) (on_board yes) (dnp no)
-    (property "Reference" "R24" (at 111.76 102.87 90)
+    (property "Reference" "R24" (at 107.315 93.345 90)
       (effects (font (size 1.27 1.27)) (justify left))
     )
-    (property "Value" "31K2" (at 114.3 103.505 90)
+    (property "Value" "31K2" (at 106.68 95.885 90)
       (effects (font (size 1.27 1.27)) (justify left))
     )
-    (property "Footprint" "Resistor_SMD:R_0402_1005Metric" (at 112.522 100.965 90)
+    (property "Footprint" "Resistor_SMD:R_0402_1005Metric" (at 109.22 94.107 90)
       (effects (font (size 1.27 1.27)) hide)
     )
-    (property "Datasheet" "~" (at 114.3 100.965 0)
+    (property "Datasheet" "~" (at 109.22 95.885 0)
       (effects (font (size 1.27 1.27)) hide)
     )
-    (property "Link" "https://www.digikey.com/en/products/detail/koa-speer-electronics-inc/RN73H1ETTP3122F25/9916907" (at 114.3 100.965 90)
+    (property "Link" "https://www.digikey.com/en/products/detail/koa-speer-electronics-inc/RN73H1ETTP3122F25/9916907" (at 109.22 95.885 90)
       (effects (font (size 1.27 1.27)) hide)
     )
-    (property "Manufacturer" "KOA Speer Electronics, Inc." (at 114.3 100.965 90)
+    (property "Manufacturer" "KOA Speer Electronics, Inc." (at 109.22 95.885 90)
       (effects (font (size 1.27 1.27)) hide)
     )
-    (property "Manufacturer Number" "RN73H1ETTP3122F25" (at 114.3 100.965 90)
+    (property "Manufacturer Number" "RN73H1ETTP3122F25" (at 109.22 95.885 90)
       (effects (font (size 1.27 1.27)) hide)
     )
-    (property "Tolerance" "1%" (at 114.3 100.965 90)
+    (property "Tolerance" "1%" (at 109.22 95.885 90)
       (effects (font (size 1.27 1.27)) hide)
     )
@@
     )
   )
-  (symbol (lib_id "Device:R") (at 109.22 95.885 270) (unit 1)
+  (symbol (lib_id "Device:R") (at 114.3 100.965 0) (unit 1)
     (in_bom yes) (on_board yes) (dnp no)
-    (property "Reference" "R8" (at 107.315 93.345 90)
+    (property "Reference" "R8" (at 111.76 102.87 90)
       (effects (font (size 1.27 1.27)) (justify left))
     )
-    (property "Value" "10K" (at 107.315 95.885 90)
+    (property "Value" "10K" (at 114.3 102.87 90)
       (effects (font (size 1.27 1.27)) (justify left))
     )
-    (property "Footprint" "Resistor_SMD:R_0402_1005Metric" (at 109.22 94.107 90)
+    (property "Footprint" "Resistor_SMD:R_0402_1005Metric" (at 112.522 100.965 90)
       (effects (font (size 1.27 1.27)) hide)
     )
-    (property "Datasheet" "https://www.koaspeer.com/pdfs/SG73P.pdf" (at 109.22 95.885 0)
+    (property "Datasheet" "https://www.koaspeer.com/pdfs/SG73P.pdf" (at 114.3 100.965 0)
       (effects (font (size 1.27 1.27)) hide)
     )
-    (property "Link" "https://www.digikey.com/en/products/detail/koa-speer-electronics-inc/SG73P1EWTTP1002F/14316756" (at 109.22 95.885 90)
+    (property "Link" "https://www.digikey.com/en/products/detail/koa-speer-electronics-inc/SG73P1EWTTP1002F/14316756" (at 114.3 100.965 90)
       (effects (font (size 1.27 1.27)) hide)
     )
-    (property "Manufacturer" "KOA Speer Electronics, Inc." (at 109.22 95.885 0)
+    (property "Manufacturer" "KOA Speer Electronics, Inc." (at 114.3 100.965 0)
       (effects (font (size 1.27 1.27)) hide)
     )
-    (property "Manufacturer Number" "SG73P1EWTTP1002F" (at 109.22 95.885 0)
+    (property "Manufacturer Number" "SG73P1EWTTP1002F" (at 114.3 100.965 0)
       (effects (font (size 1.27 1.27)) hide)
     )
-    (property "Notes" "DNP" (at 109.22 95.885 0)
+    (property "Notes" "DNP" (at 114.3 100.965 0)
       (effects (font (size 1.27 1.27)) hide)
     )
@@
     )
   )
-  (symbol (lib_id "Device:R") (at 182.88 100.965 180) (unit 1)
+  (symbol (lib_id "Device:R") (at 187.96 95.885 90) (unit 1)
     (in_bom yes) (on_board yes) (dnp no)
-    (property "Reference" "R26" (at 185.42 99.06 90)
+    (property "Reference" "R26" (at 189.865 93.345 90)
       (effects (font (size 1.27 1.27)) (justify left))
     )
-    (property "Value" "52K3" (at 182.88 98.425 90)
+    (property "Value" "52K3" (at 190.5 95.885 90)
       (effects (font (size 1.27 1.27)) (justify left))
     )
-    (property "Footprint" "Resistor_SMD:R_0402_1005Metric" (at 184.658 100.965 90)
+    (property "Footprint" "Resistor_SMD:R_0402_1005Metric" (at 187.96 97.663 90)
       (effects (font (size 1.27 1.27)) hide)
     )
-    (property "Datasheet" "~" (at 182.88 100.965 0)
+    (property "Datasheet" "~" (at 187.96 95.885 0)
       (effects (font (size 1.27 1.27)) hide)
     )
-    (property "Manufacturer Number" "RT0402FRE0752K3L" (at 182.88 100.965 90)
+    (property "Manufacturer Number" "RT0402FRE0752K3L" (at 187.96 95.885 90)
       (effects (font (size 1.27 1.27)) hide)
     )
-    (property "Tolerance" "1%" (at 182.88 100.965 90)
+    (property "Tolerance" "1%" (at 187.96 95.885 90)
       (effects (font (size 1.27 1.27)) hide)
     )
-    (property "Link" "https://www.digikey.com/en/products/detail/yageo/RT0402FRE0752K3L/1072062" (at 182.88 100.965 90)
+    (property "Link" "https://www.digikey.com/en/products/detail/yageo/RT0402FRE0752K3L/1072062" (at 187.96 95.885 90)
       (effects (font (size 1.27 1.27)) hide)
     )
-    (property "Manufacturer" "Yageo" (at 182.88 100.965 90)
+    (property "Manufacturer" "Yageo" (at 187.96 95.885 90)
       (effects (font (size 1.27 1.27)) hide)
     )
