File: hardware/ttl_io/power_supplies.kicad_sch (KiCad schematic)
At the start: 23 parts, among them J4 Barrel_Jack_Switch, U8 LT3506

Commit message: draft pcb v0.1.0
Parts:
- J4: footprint Connector_BarrelJack:BarrelJack_CUI_PJ-036AH-SMT_Horizontal -> Connector_BarrelJack:BarrelJack_CUI_PJ-102AH_Horizontal; Link https://www.digikey.com/en/products/detail/cui-devices/PJ-0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 -> https://www.digikey.com/en/products/detail/cui-devices/PJ-1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; Manufacturer Number PJ-036AH-SMT-TR -> PJ-102AH; PCBWay Link https://www.pcbway.com/components/detail/PJ036AHSMTTR/39245/ -> https://www.pcbway.com/components/detail/PJ102AH/484087/
Changed lines of the file:
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@@
-    )
-  )
-  (symbol (lib_id "Connector:Barrel_Jack_Switch") (at 29.845 69.85 0) (unit 1)
-    (in_bom yes) (on_board yes) (dnp no)
-    (property "Reference" "J4" (at 26.035 64.77 0)
-      (effects (font (size 1.27 1.27)))
-    )
-    (property "Value" "Barrel_Jack_Switch" (at 29.845 63.5 0)
-      (effects (font (size 1.27 1.27)) hide)
-    )
-    (property "Footprint" "Connector_BarrelJack:BarrelJack_CUI_PJ-036AH-SMT_Horizontal" (at 31.115 70.866 0)
-      (effects (font (size 1.27 1.27)) hide)
-    )
-    (property "Datasheet" "https://www.cuidevices.com/product/resource/pj-036ah-smt-tr.pdf" (at 31.115 70.866 0)
-      (effects (font (size 1.27 1.27)) hide)
-    )
-    (property "Link" "https://www.digikey.com/en/products/detail/cui-devices/PJ-036AH-SMT-TR/1530994?" (at 29.845 69.85 0)
-      (effects (font (size 1.27 1.27)) hide)
-    )
-    (property "Manufacturer Number" "PJ-036AH-SMT-TR" (at 29.845 69.85 0)
-      (effects (font (size 1.27 1.27)) hide)
-    )
-    (property "PCBWay Link" "https://www.pcbway.com/components/detail/PJ036AHSMTTR/39245/" (at 29.845 69.85 0)
-      (effects (font (size 1.27 1.27)) hide)
-    )
-    (property "Manufacturer" "CUI Devices" (at 29.845 69.85 0)
-      (effects (font (size 1.27 1.27)) hide)
-    )
-    (pin "1")
-    (pin "2")
-    (pin "3")
-    (instances
-      (project "ttl_io"
-        (path "/de782c9d-fd54-45ed-aa91-6297331e40f6/76bb2607-2d2e-4d2c-9a45-1b3b3938988a"
-          (reference "J4") (unit 1)
-        )
-      )
-      (project "harp_lick_detector_capactive"
-        (path "/e63e39d7-6ac0-4ffd-8aa3-1841a4541b55"
-          (reference "J5") (unit 1)
-        )
-        (path "/e63e39d7-6ac0-4ffd-8aa3-1841a4541b55/b51b21ef-b374-4f9f-a058-7db9b64fdf4a"
-          (reference "J6") (unit 1)
-        )
-      )
     )
   )
@@
         )
       )
+    )
+  )
+  (symbol (lib_id "Connector:Barrel_Jack_Switch") (at 29.845 69.85 0) (unit 1)
+    (in_bom yes) (on_board yes) (dnp no)
+    (property "Reference" "J4" (at 26.035 64.77 0)
+      (effects (font (size 1.27 1.27)))
+    )
+    (property "Value" "Barrel_Jack_Switch" (at 29.845 63.5 0)
+      (effects (font (size 1.27 1.27)) hide)
+    )
+    (property "Footprint" "Connector_BarrelJack:BarrelJack_CUI_PJ-102AH_Horizontal" (at 31.115 70.866 0)
+      (effects (font (size 1.27 1.27)) hide)
+    )
+    (property "Datasheet" "https://www.cuidevices.com/product/resource/pj-102ah.pdf" (at 31.115 70.866 0)
+      (effects (font (size 1.27 1.27)) hide)
+    )
+    (property "Link" "https://www.digikey.com/en/products/detail/cui-devices/PJ-102AH/408448" (at 29.845 69.85 0)
+      (effects (font (size 1.27 1.27)) hide)
+    )
+    (property "Manufacturer Number" "PJ-102AH" (at 29.845 69.85 0)
+      (effects (font (size 1.27 1.27)) hide)
+    )
+    (property "PCBWay Link" "https://www.pcbway.com/components/detail/PJ102AH/484087/" (at 29.845 69.85 0)
+      (effects (font (size 1.27 1.27)) hide)
+    )
+    (property "Manufacturer" "CUI Devices" (at 29.845 69.85 0)
+      (effects (font (size 1.27 1.27)) hide)
+    )
+    (pin "1")
+    (pin "2")
+    (pin "3")
+    (instances
+      (project "ttl_io"
+        (path "/de782c9d-fd54-45ed-aa91-6297331e40f6/76bb2607-2d2e-4d2c-9a45-1b3b3938988a"
+          (reference "J4") (unit 1)
+        )
+      )
+      (project "harp_lick_detector_capactive"
+        (path "/e63e39d7-6ac0-4ffd-8aa3-1841a4541b55"
+          (reference "J5") (unit 1)
+        )
+        (path "/e63e39d7-6ac0-4ffd-8aa3-1841a4541b55/b51b21ef-b374-4f9f-a058-7db9b64fdf4a"
+          (reference "J6") (unit 1)
+        )
+      )

Commit message: update pcb and bom
Parts:
- D6, D7, D8: Manufacturer (none) -> SMC Diode Solutions
Changed lines of the file:
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@@
+      (effects (font (size 1.27 1.27)) hide)
+    )
+    (property "Manufacturer" "SMC Diode Solutions" (at 178.435 100.965 0)
       (effects (font (size 1.27 1.27)) hide)
     )
@@
     )
     (property "Manufacturer Number" "MBR260HW" (at 119.38 100.965 0)
+      (effects (font (size 1.27 1.27)) hide)
+    )
+    (property "Manufacturer" "SMC Diode Solutions" (at 119.38 100.965 0)
       (effects (font (size 1.27 1.27)) hide)
     )
@@
       (effects (font (size 1.27 1.27)) hide)
     )
+    (property "Manufacturer" "SMC Diode Solutions" (at 50.8 67.31 0)
+      (effects (font (size 1.27 1.27)) hide)
+    )

Commit message: add hw/fw licenses
Parts:
- C36, C38: Manufacturer (none) -> Samsung Electro-Mechanics
- L2, L3: Manufacturer (none) -> Vishay Dale; Manufacturer Number (none) -> IHLP2525CZER100M11
Changed lines of the file:
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@@
       (effects (font (size 1.27 1.27)) hide)
     )
-    (property "Datasheet" "~" (at 129.54 95.885 0)
+    (property "Datasheet" "https://www.yageo.com/upload/media/product/app/datasheet/mlcc/upy-gphc_x7r_6_3v-to-250v.pdf" (at 129.54 95.885 0)
       (effects (font (size 1.27 1.27)) hide)
     )
@@
     )
     (property "PCBWay Link" "todo" (at 101.6 100.965 0)
+      (effects (font (size 1.27 1.27)) hide)
+    )
+    (property "Manufacturer" "Samsung Electro-Mechanics" (at 101.6 100.965 0)
       (effects (font (size 1.27 1.27)) hide)
     )
@@
       (effects (font (size 1.27 1.27)) hide)
     )
-    (property "Datasheet" "~" (at 178.435 100.965 0)
+    (property "Datasheet" "https://www.smc-diodes.com/propdf/MBR260HW%20N1503%20REV.B.pdf" (at 178.435 100.965 0)
       (effects (font (size 1.27 1.27)) hide)
     )
@@
       (effects (font (size 1.27 1.27)) hide)
     )
-    (property "Datasheet" "~" (at 119.38 100.965 0)
+    (property "Datasheet" "https://www.smc-diodes.com/propdf/MBR260HW%20N1503%20REV.B.pdf" (at 119.38 100.965 0)
       (effects (font (size 1.27 1.27)) hide)
     )
@@
       (effects (font (size 1.27 1.27)) hide)
     )
-    (property "Datasheet" "~" (at 112.395 90.805 0)
+    (property "Datasheet" "https://www.vishay.com/docs/34190/ihlp-2525cz-11.pdf" (at 112.395 90.805 0)
       (effects (font (size 1.27 1.27)) hide)
     )
     (property "Link" "https://www.digikey.com/en/products/detail/vishay-dale/IHLP2525CZER100M11/1220685" (at 112.395 90.805 90)
+      (effects (font (size 1.27 1.27)) hide)
+    )
+    (property "Manufacturer" "Vishay Dale" (at 112.395 90.805 0)
+      (effects (font (size 1.27 1.27)) hide)
+    )
+    (property "Manufacturer Number" "IHLP2525CZER100M11" (at 112.395 90.805 0)
       (effects (font (size 1.27 1.27)) hide)
     )
@@
       (effects (font (size 1.27 1.27)) hide)
     )
-    (property "Datasheet" "~" (at 167.64 95.885 0)
+    (property "Datasheet" "https://www.yageo.com/upload/media/product/app/datasheet/mlcc/upy-gphc_x7r_6_3v-to-250v.pdf" (at 167.64 95.885 0)
       (effects (font (size 1.27 1.27)) hide)
     )
@@
       (effects (font (size 1.27 1.27)) hide)
     )
-    (property "Datasheet" "~" (at 109.22 95.885 0)
+    (property "Datasheet" "https://www.koaspeer.com/pdfs/RN73H.pdf" (at 109.22 95.885 0)
       (effects (font (size 1.27 1.27)) hide)
     )
@@
       (effects (font (size 1.27 1.27)) hide)
     )
-    (property "Datasheet" "~" (at 184.15 90.805 0)
+    (property "Datasheet" "https://www.vishay.com/docs/34190/ihlp-2525cz-11.pdf" (at 184.15 90.805 0)
       (effects (font (size 1.27 1.27)) hide)
     )
@@
       (effects (font (size 1.27 1.27)) hide)
     )
+    (property "Manufacturer" "Vishay Dale" (at 184.15 90.805 0)
+      (effects (font (size 1.27 1.27)) hide)
+    )
+    (property "Manufacturer Number" "IHLP2525CZER100M11" (at 184.15 90.805 0)
+      (effects (font (size 1.27 1.27)) hide)
+    )
     (pin "1")
     (pin "2")
@@
       (effects (font (size 1.27 1.27)) hide)
     )
-    (property "Datasheet" "~" (at 187.96 95.885 0)
+    (property "Datasheet" "https://www.yageo.com/upload/media/product/app/datasheet/rchip/pyu-rt_1-to-0.01_rohs_l.pdf" (at 187.96 95.885 0)
       (effects (font (size 1.27 1.27)) hide)
     )
@@
       (effects (font (size 1.27 1.27)) hide)
     )
+    (property "Manufacturer" "Samsung Electro-Mechanics" (at 194.945 100.965 0)
+      (effects (font (size 1.27 1.27)) hide)
+    )
     (pin "1")
     (pin "2")
@@
       (effects (font (size 1.27 1.27)) hide)
     )
-    (property "Datasheet" "~" (at 50.8 67.31 0)
-      (effects (font (size 1.27 1.27)) hide)
-    )
+    (property "Datasheet" "https://www.smc-diodes.com/propdf/MBR260HW%20N1503%20REV.B.pdf" (at 50.8 67.31 0)
+      (effects (font (size 1.27 1.27)) hide)
+    )

Commit message: get pwm task and ios working
Parts:
- renumbered C6 to C31, C6 to C32, R8 to R21, R8 to R22, R8 to R23, R8 to R25
Changed lines of the file:
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@@
   (symbol (lib_id "Device:C") (at 178.435 85.725 0) (mirror x) (unit 1)
     (in_bom yes) (on_board yes) (dnp no)
-    (property "Reference" "C6" (at 173.99 83.185 0)
+    (property "Reference" "C32" (at 173.99 83.185 0)
       (effects (font (size 1.27 1.27)) (justify left))
     )
@@
     (instances
       (project "ttl_io"
-        (path "/de782c9d-fd54-45ed-aa91-6297331e40f6/1fe1f8ff-b1f9-48b6-8256-97b16d4120ca"
-          (reference "C6") (unit 1)
-        )
         (path "/de782c9d-fd54-45ed-aa91-6297331e40f6/76bb2607-2d2e-4d2c-9a45-1b3b3938988a"
           (reference "C32") (unit 1)
@@
   (symbol (lib_id "Device:C") (at 119.38 85.725 180) (unit 1)
     (in_bom yes) (on_board yes) (dnp no)
-    (property "Reference" "C6" (at 123.825 83.185 0)
+    (property "Reference" "C31" (at 123.825 83.185 0)
       (effects (font (size 1.27 1.27)) (justify left))
     )
@@
     (instances
       (project "ttl_io"
-        (path "/de782c9d-fd54-45ed-aa91-6297331e40f6/1fe1f8ff-b1f9-48b6-8256-97b16d4120ca"
-          (reference "C6") (unit 1)
-        )
         (path "/de782c9d-fd54-45ed-aa91-6297331e40f6/76bb2607-2d2e-4d2c-9a45-1b3b3938988a"
           (reference "C31") (unit 1)
@@
   (symbol (lib_id "Device:R") (at 182.88 100.965 180) (unit 1)
     (in_bom yes) (on_board yes) (dnp no)
-    (property "Reference" "R8" (at 185.42 99.06 90)
+    (property "Reference" "R25" (at 185.42 99.06 90)
       (effects (font (size 1.27 1.27)) (justify left))
     )
@@
     (instances
       (project "ttl_io"
-        (path "/de782c9d-fd54-45ed-aa91-6297331e40f6/1fe1f8ff-b1f9-48b6-8256-97b16d4120ca"
-          (reference "R8") (unit 1)
-        )
         (path "/de782c9d-fd54-45ed-aa91-6297331e40f6/76bb2607-2d2e-4d2c-9a45-1b3b3938988a"
           (reference "R25") (unit 1)
@@
   (symbol (lib_id "Device:R") (at 172.72 100.965 0) (mirror x) (unit 1)
     (in_bom yes) (on_board yes) (dnp no)
-    (property "Reference" "R8" (at 173.355 97.155 0)
+    (property "Reference" "R23" (at 173.355 97.155 0)
       (effects (font (size 1.27 1.27)) (justify left))
     )
@@
     (instances
       (project "ttl_io"
-        (path "/de782c9d-fd54-45ed-aa91-6297331e40f6/1fe1f8ff-b1f9-48b6-8256-97b16d4120ca"
-          (reference "R8") (unit 1)
-        )
         (path "/de782c9d-fd54-45ed-aa91-6297331e40f6/76bb2607-2d2e-4d2c-9a45-1b3b3938988a"
           (reference "R23") (unit 1)
@@
   (symbol (lib_id "Device:R") (at 124.46 100.965 180) (unit 1)
     (in_bom yes) (on_board yes) (dnp no)
-    (property "Reference" "R8" (at 123.825 97.155 0)
+    (property "Reference" "R22" (at 123.825 97.155 0)
       (effects (font (size 1.27 1.27)) (justify left))
     )
@@
     (instances
       (project "ttl_io"
-        (path "/de782c9d-fd54-45ed-aa91-6297331e40f6/1fe1f8ff-b1f9-48b6-8256-97b16d4120ca"
-          (reference "R8") (unit 1)
-        )
         (path "/de782c9d-fd54-45ed-aa91-6297331e40f6/76bb2607-2d2e-4d2c-9a45-1b3b3938988a"
           (reference "R22") (unit 1)
@@
   (symbol (lib_id "Device:R") (at 114.3 100.965 0) (unit 1)
     (in_bom yes) (on_board yes) (dnp no)
-    (property "Reference" "R8" (at 111.76 102.87 90)
+    (property "Reference" "R21" (at 111.76 102.87 90)
       (effects (font (size 1.27 1.27)) (justify left))
     )
@@
     (instances
       (project "ttl_io"
-        (path "/de782c9d-fd54-45ed-aa91-6297331e40f6/1fe1f8ff-b1f9-48b6-8256-97b16d4120ca"
-          (reference "R8") (unit 1)
-        )
         (path "/de782c9d-fd54-45ed-aa91-6297331e40f6/76bb2607-2d2e-4d2c-9a45-1b3b3938988a"
           (reference "R21") (unit 1)
